File: PCB/Main/Main.kicad_pcb (KiCad board)
At the start: 2 copper layers, 0 parts

Commit message: rename y conectores
tambien se añaden pours
Parts:
- added J1: HDMI_A_1.4, Connector_Video:HDMI_A_Molex_208658-1001_Horizontal, F.Cu at (55.5, 97.3)
- added J2: Conn_01x02_Pin, TerminalBlock_Phoenix:TerminalBlock_Phoenix_PT-1,5-2-5.0-H_1x02_P5.00mm_Horizontal, F.Cu at (148.7, 72.8)
- added J3: Conn_01x01, Connector_PinHeader_2.54mm:PinHeader_1x01_P2.54mm_Horizontal, F.Cu at (148.0, 53.3)
- added J4: Conn_02x04_Odd_Even, Connector_PinHeader_2.54mm:PinHeader_2x04_P2.54mm_Horizontal, F.Cu at (148.0, 55.5)
- added J5: Conn_01x06, Connector_PinHeader_2.54mm:PinHeader_1x06_P2.54mm_Horizontal, F.Cu at (134.1, 57.9)
- added U1: ORANGE_PI_CM4, Footprint:OCM4, F.Cu at (62.0, 50.5)
- added U2: ESD224DQA, Package_DFN_QFN:Diodes_UDFN-10_1x2.5mm_P0.5mm, F.Cu at (58.5, 84.1)
- added U3: ESD224DQA, Package_DFN_QFN:Diodes_UDFN-10_1x2.5mm_P0.5mm, F.Cu at (54.5, 83.0)
- added U4: ESD224DQA, Package_DFN_QFN:Diodes_UDFN-10_1x2.5mm_P0.5mm, F.Cu at (48.5, 74.4)
Routing:
- net GND: track 0.00 -> 12.7 mm, vias 0 -> 5
- net /JP2/HDMI0_D2_IN_P: track 0.00 -> 4.13 mm
- net /JP2/HDMI0_D2_IN_N: track 0.00 -> 4.13 mm
- net +5V: track 0.00 -> 2.71 mm, vias 0 -> 1
- added copper zone on B.Cu, net (none)
- added copper zone on In2.Cu, net +3.3V
- added copper zone on In2.Cu, net +5V
- added copper zone on F.Cu, net GND
- added copper zone on In1.Cu, net GND
Other:
- copper layers 2 -> 4

Commit message: pcb continued
Parts:
- added C1: 470µF, Capacitor_Tantalum_SMD:CP_EIA-7343-31_Kemet-D, F.Cu at (23.5, 27.6)
- added C2: 100nF, Capacitor_SMD:C_0603_1608Metric, F.Cu at (23.3, 53.5)
- moved J2 130.1 mm to (22.4, 41.5), turned to 90 degrees
- moved J5 119.7 mm to (20.4, 20.7), turned to 90 degrees
- moved J4 37.4 mm to (122.0, 82.4)
- moved J3 25.6 mm to (123.1, 47.5)
Connections:
- J2 pad 2: GND -> /Power/POWER_GND
- J5 pad 1: GND -> /Power/POWER_GND
- J5 pad 4: /Power/EN -> /JP1/EN
- J5 pad 5: GND -> /Power/POWER_GND
- J5 pad 6: /Power/VOUT -> /Power/POWER_5V
- U1 pad JP1_1: unconnected-(U1A-GND_JP1_1-PadJP1_1) -> GND
- U1 pad JP1_13: unconnected-(U1A-GND_JP1_13-PadJP1_13) -> GND
- U1 pad JP1_14: unconnected-(U1A-GND_JP1_14-PadJP1_14) -> GND
- U1 pad JP1_2: unconnected-(U1A-GND_JP1_2-PadJP1_2) -> GND
- U1 pad JP1_22: unconnected-(U1A-GND_JP1_22-PadJP1_22) -> GND
- U1 pad JP1_23: unconnected-(U1A-GND_JP1_23-PadJP1_23) -> GND
- U1 pad JP1_32: unconnected-(U1A-GND_JP1_32-PadJP1_32) -> GND
- U1 pad JP1_33: unconnected-(U1A-GND_JP1_33-PadJP1_33) -> GND
- U1 pad JP1_42: unconnected-(U1A-GND_JP1_42-PadJP1_42) -> GND
- U1 pad JP1_43: unconnected-(U1A-GND_JP1_43-PadJP1_43) -> GND
- U1 pad JP1_52: unconnected-(U1A-GND_JP1_52-PadJP1_52) -> GND
- U1 pad JP1_53: unconnected-(U1A-GND_JP1_53-PadJP1_53) -> GND
- U1 pad JP1_59: unconnected-(U1A-GND_JP1_59-PadJP1_59) -> GND
- U1 pad JP1_60: unconnected-(U1A-GND_JP1_60-PadJP1_60) -> GND
- U1 pad JP1_65: unconnected-(U1A-GND_JP1_65-PadJP1_65) -> GND
- U1 pad JP1_66: unconnected-(U1A-GND_JP1_66-PadJP1_66) -> GND
- U1 pad JP1_7: unconnected-(U1A-GND_JP1_7-PadJP1_7) -> GND
- U1 pad JP1_71: unconnected-(U1A-GND_JP1_71-PadJP1_71) -> GND
- U1 pad JP1_74: unconnected-(U1A-GND_JP1_74-PadJP1_74) -> GND
- U1 pad JP1_77: unconnected-(U1A-VBUS_JP1_77-PadJP1_77) -> +5V
- U1 pad JP1_79: unconnected-(U1A-VBUS_JP1_79-PadJP1_79) -> +5V
- U1 pad JP1_8: unconnected-(U1A-GND_JP1_8-PadJP1_8) -> GND
- U1 pad JP1_81: unconnected-(U1A-VBUS_JP1_81-PadJP1_81) -> +5V
- U1 pad JP1_83: unconnected-(U1A-VBUS_JP1_83-PadJP1_83) -> +5V
- U1 pad JP1_85: unconnected-(U1A-VBUS_JP1_85-PadJP1_85) -> +5V
- U1 pad JP1_87: unconnected-(U1A-VBUS_JP1_87-PadJP1_87) -> +5V
- U1 pad JP1_98: unconnected-(U1A-GND_JP1_98-PadJP1_98) -> GND
- U1 pad JP1_99: unconnected-(U1A-PMIC_PWRON-PadJP1_99) -> /JP1/EN
Routing:
- net GND: track 12.7 -> 65.9 mm
- net /JP1/EN: track 0.00 -> 36.0 mm
- net /Power/POWER_GND: track 0.00 -> 12.6 mm, vias 0 -> 5
- net /Power/POWER_5V: track 0.00 -> 7.69 mm, vias 0 -> 3
- net +5V: track 2.71 -> 7.41 mm
- added copper zone on F.Cu, net +5V
- added copper zone on F.Cu, net /Power/POWER_5V
- added copper zone on F.Cu, net /Power/POWER_GND

Commit message: pitty
Parts:
- added J6: USB_A, Connector_USB:USB_A_Molex_67643_Horizontal, F.Cu at (26.8, 128.3)
- added J7: USB3_A, Connector_USB:USB3_A_Molex_48393-001, F.Cu at (25.9, 164.3)
- added J8: USB_A, Connector_USB:USB_A_Molex_67643_Horizontal, F.Cu at (26.9, 146.4)
Connections:
- U1 pad JP3_1: unconnected-(U1C-GND_JP3_1-PadJP3_1) -> GND
- U1 pad JP3_11: unconnected-(U1C-USB2_HOST2_DP-PadJP3_11) -> Net-(J8-D+)
- U1 pad JP3_13: unconnected-(U1C-GND_JP3_13-PadJP3_13) -> GND
- U1 pad JP3_14: unconnected-(U1C-GND_JP3_14-PadJP3_14) -> GND
- U1 pad JP3_16: unconnected-(U1C-USB3_HOST1_SSTXN-PadJP3_16) -> Net-(U1C-USB3_HOST1_SSTXN)
- U1 pad JP3_17: unconnected-(U1C-GND_JP3_17-PadJP3_17) -> GND
- U1 pad JP3_18: unconnected-(U1C-USB3_HOST1_SSTXP-PadJP3_18) -> Net-(U1C-USB3_HOST1_SSTXP)
- U1 pad JP3_19: unconnected-(U1C-USB3_HOST1_DM-PadJP3_19) -> Net-(J7-D-)
- U1 pad JP3_2: unconnected-(U1C-GND_JP3_2-PadJP3_2) -> GND
- U1 pad JP3_20: unconnected-(U1C-GND_JP3_20-PadJP3_20) -> GND
- U1 pad JP3_21: unconnected-(U1C-USB3_HOST1_DP-PadJP3_21) -> Net-(J7-D+)
- U1 pad JP3_22: unconnected-(U1C-USB3_HOST1_SSRXP-PadJP3_22) -> Net-(J7-SSTX+)
- U1 pad JP3_23: unconnected-(U1C-GND_JP3_23-PadJP3_23) -> GND
- U1 pad JP3_24: unconnected-(U1C-USB3_HOST1_SSRXN-PadJP3_24) -> Net-(J7-SSTX-)
- U1 pad JP3_3: unconnected-(U1C-USB2_HOST3_DM-PadJP3_3) -> Net-(J6-D-)
- U1 pad JP3_5: unconnected-(U1C-USB2_HOST3_DP-PadJP3_5) -> Net-(J6-D+)
- U1 pad JP3_7: unconnected-(U1C-GND_JP3_7-PadJP3_7) -> GND
- U1 pad JP3_9: unconnected-(U1C-USB2_HOST2_DM-PadJP3_9) -> Net-(J8-D-)
